Commit message: camera frame corrected

File: Project 4/my_robot/urdf/my_robot.xacro (robot description, xacro)
@@ -14,6 +14,6 @@
   </gazebo>
 !--...............................LINKS.................................................-->
+  <link name="robot_footprint"></link>
   <xacro:include filename="$(find my_robot)/urdf/my_robot.gazebo" />
-  <link name="robot_footprint"></link>
 <!-- Link details for chassis-->
   <link name='chassis'>
@@ -115,7 +115,8 @@
   <!-- Link details for Camera-->
   <link name="camera">
+    <pose> 0 0 0 0 0 0 </pose>
     <inertial>
       <mass value="0.1"/>
-      <origin xyz="0.0 0.0 0.0" rpy="0 0 0"/>
+      <origin xyz="0.0 0.0 0.0" rpy="0.0 0 0"/>
       <inertia
         ixx="1e-6" ixy="0.0" ixz="0.0"
@@ -139,4 +140,5 @@
   <!-- Link details for LIDAR-->
   <link name="hokuyo">
+  <pose> 0 0 0 0 0 </pose>
     <inertial>
       <mass value="1e-5"/>
@@ -197,8 +199,10 @@
     <parent link="chassis"/>
     <child link="hokuyo" />
-    <axis xyz="0 1 0"/>
+    <axis xyz="0 1 0" rpy = "0 0 0"/>
+    <limit effort="10000" velocity="1000"/>
+    <dynamics dampning="1.0" friction="1.0"/>
   </joint>
   <joint name="camera_optical_joint" type="fixed">
-    <origin xyz="0 0 0" rpy="-1.5707 0 -1.5707"/>
+    <origin xyz="0 0 0" rpy="0 0 0"/>
     <parent link="camera"/>
     <child link="camera_link_optical"/>

Commit message: Point cloud frame corrected and map generated

File: Project 4/my_robot/urdf/my_robot.xacro (robot description, xacro)
@@ -204,5 +204,5 @@
   </joint>
   <joint name="camera_optical_joint" type="fixed">
-    <origin xyz="0 0 0" rpy="0 0 0"/>
+    <origin xyz="0 0 0" rpy="-1.5707 0 -1.5707"/>
     <parent link="camera"/>
     <child link="camera_link_optical"/>
